File: board/board.kicad_sch (KiCad schematic)
At the start: 21 parts

Commit message: updated schematic
Parts:
- removed U?: TFT_Touch_Shield_WaveShare, symbol ownLib:TFT_Touch_Shield_WaveShare
- added J?: Display, symbol Connector_Generic:Conn_01x20
- added U?: PCF8574, symbol Interface_Expansion:PCF8574
- TP?: value G4 -> G2
Connections:
- net +3V3: now also J?.3 (Pin_3); no longer R?.1, R?.1
- net +5V: now also J?.2 (Pin_2)
- net GND: now also J?.1 (Pin_1), J?.15 (Pin_15)
- net HSPI_CS: now also J?.7 (Pin_7)
- net HSPI_MISO: now also J?.5 (Pin_5)
- net HSPI_MOSI: now also J?.6 (Pin_6)
- net HSPI_SCK: now also J?.4 (Pin_4)
- net LCD_BL: now also J?.10 (Pin_10)
- net LCD_DC: now also J?.8 (Pin_8)
- net LCD_RST: now also J?.9 (Pin_9)
- net TOUCH_X+: now also J?.12 (Pin_12)
- net TOUCH_X-: now also J?.14 (Pin_14)
- net TOUCH_Y+: now also J?.11 (Pin_11)
- net TOUCH_Y-: now also J?.13 (Pin_13)
- net SIG_SW: now reaches U?.10 (IO26)
- new net 3V3_SW: R?.1, R?.1
- no-connect marks 12 -> 15
Other:
- sheet IMU ports: added 3V3; removed none
- sheet PowerSupply ports: added 3V3SW, 5VSW, SIG_SW; removed none
- sheet Pulsoxymeter ports: added 3V3, 5V; removed none
- note added: "TODO: IO-Extender?"
- note removed: "TODO: I2C devices with MOSFET on switched pwrsupply"
- moved on the sheet: U?
