File: board/board.kicad_pcb (KiCad board)
At the start: 2 copper layers, 160 x 120 mm, 167 parts, among them J1 Display, J10 Analog CH1, J11 Analog CH2, J12 Analog CH3, J13 Analog CH4, J14 Analog CH5, J15 Micro_SD_Card, J16 OXY, J17 I2C, J18 SPI, J19 GPIO, J2 BIAS, J20 3V3, J21 GND, J22 5V, J3 SRB, J4 EEG Out, J5 Device Electrodes, J6 REF, J7 Analog CH6, J8 Analog CH7, J9 Analog CH0, Q1 BSH203,215, Q2 BSH203,215, Q3 BSH203,215, Q4 BSH203,215, Q5 BSH203,215, SW1 MAIN, U1 ESP32-DevKitC, U10 TLV840C, U11 PCF8574, U2 ADS1299-x, U3 BHI160, U4 MCP3564RT, U5 LM1117-5.0, U6 NCV8165, U7 NCP115, U8 MIC5209, U9 NUF6401, X1 ECS-2520MVLC-020.48-BN-TR

Commit message: WIP pushed for meeting
Parts:
- added C50: 100n, Capacitor_SMD:C_0402_1005Metric, F.Cu at (6.60, 53.9)
- added JP13: A0, Jumper:SolderJumper-3_P1.3mm_Bridged12_Pad1.0x1.5mm, F.Cu at (7.90, 58.5)
- added JP14: A1, Jumper:SolderJumper-3_P1.3mm_Bridged12_Pad1.0x1.5mm, F.Cu at (4.40, 54.6)
- added TP29: IN1, TestPoint:TestPoint_Pad_D1.0mm, F.Cu at (14.1, 58.3)
- added TP30: IN2, TestPoint:TestPoint_Pad_D1.0mm, F.Cu at (11.8, 58.3)
- added U12: TSC2003, ownLib:TSSOP-16_4.4x5mm_P0.65mm_EP3x3mm, F.Cu at (9.90, 51.4)
- C6: value 1u -> 100n; footprint Capacitor_SMD:C_0603_1608Metric -> Capacitor_SMD:C_0402_1005Metric
- TP18: value MCLKIN -> MCLK
- U4: footprint ownLib:HTSSOP-20-1EP_4.4x6.5mm_P0.65mm_3.4x6.5mm_Mask2.75x3.43mm -> Package_SO:HTSSOP-20-1EP_4.4x6.5mm_P0.65mm_EP3.4x6.5mm_Mask2.75x3.43mm
- moved R4 208.9 mm to (133.4, 18.6), turned to 180 degrees
- moved TP12 197.8 mm to (130.6, 15.0)
- moved C48 185.3 mm to (116.5, 41.9), turned to 180 degrees
- moved C49 184.0 mm to (116.9, 43.2), turned to 180 degrees
- moved R3 168.9 mm to (112.2, 65.0), turned to 180 degrees
- moved TP13 166.1 mm to (109.8, 65.2)
- moved TP15 163.2 mm to (104.0, 68.8)
- moved FB1 162.4 mm to (139.1, 25.3), turned to -90 degrees
- moved TP16 161.7 mm to (105.5, 67.3)
- moved TP14 161.6 mm to (105.5, 70.3)
- moved TP17 151.0 mm to (104.0, 65.8)
- moved C33 147.0 mm to (137.8, 25.0), turned to 90 degrees
- moved C29 146.2 mm to (130.9, 25.3), turned to 90 degrees
- moved C31 143.5 mm to (136.5, 25.3), turned to 90 degrees
- moved TP4 142.6 mm to (80.8, 46.8)
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Connections:
- C19 pad 1: +3V3 -> /3V3_SW
- C20 pad 1: +3V3 -> /3V3_SW
- C6 pad 1: AVSS -> /3V3_SW
- J1 pad 10: /LCD_BL -> /LCD_RST
- J1 pad 11: /TOUCH_Y+ -> Net-(J1-Pad11)
- J1 pad 12: /TOUCH_X+ -> Net-(J1-Pad12)
- J1 pad 13: /TOUCH_Y- -> Net-(J1-Pad13)
- J1 pad 14: /TOUCH_X- -> Net-(J1-Pad14)
- J1 pad 9: /LCD_RST -> /LCD_BL
- JP5 pad 1: /EKG/EEGMux/IN3N_OUT -> /EKG/EEGMux/IN2N_OUT
- JP6 pad 1: /EKG/EEGMux/IN2N_OUT -> /EKG/EEGMux/IN3N_OUT
- JP8 pad 3: +3V3 -> /3V3_SW
- TP18 pad 1: /ADC/MCLK -> /MCLK
- U1 pad 10: /SIG_SW -> /LCD_RST
- U1 pad 11: /TOUCH_X- -> /SIG_SW
- U1 pad 32: /TOUCH_Y+ -> /~{EKGReset}
- U1 pad 33: /TOUCH_Y- -> /~{EKGPowerDown}
- U1 pad 34: /TOUCH_X+ -> /~{DISPLAY_IRQ}
- U1 pad 8: /~{EKGReset} -> /LCD_BL
- U1 pad 9: /~{EKGPowerDown} -> /LCD_DC
- U3 pad 8: +3V3 -> /3V3_SW
Routing:
- net +3V3: track 0.00 -> 386.0 mm, vias 0 -> 12
- net /VSPI_SCK: track 0.00 -> 277.7 mm, vias 0 -> 5
- net /VSPI_MOSI: track 0.00 -> 276.0 mm, vias 0 -> 4
- net /VSPI_MISO: track 0.00 -> 273.7 mm, vias 0 -> 4
- net /I2C1_SDA: track 0.00 -> 256.4 mm, vias 0 -> 3
- net /I2C1_SCK: track 0.00 -> 249.3 mm, vias 0 -> 3
- net +5V: track 0.00 -> 198.7 mm, vias 0 -> 3
- net +6V: track 0.00 -> 147.7 mm, vias 0 -> 5
- net /~{ADC_INT}: track 0.00 -> 143.0 mm, vias 0 -> 1
- net /3V3_SW: track 0.00 -> 140.8 mm, vias 0 -> 14
- net /ADC_CS: track 0.00 -> 111.5 mm, vias 0 -> 1
- net +3.3VA: track 0.00 -> 76.5 mm, vias 0 -> 1
- net /EKG/EEGMux/BIAS: track 0.00 -> 69.0 mm
- net /~{SDPowerOK}: track 0.00 -> 66.1 mm, vias 0 -> 1
- net /MCLK: track 0.00 -> 62.6 mm
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- added copper zone on B.Cu, net AVSS
- added copper zone on F.Cu, net AVSS
- added copper zone on In1.Cu, net AVSS
- added copper zone on In2.Cu, net AVSS
Other:
- board size 160 x 120 mm -> 160 x 95 mm
- copper layers 2 -> 4
