File: board/board.kicad_pcb (KiCad board)
At the start: 4 copper layers, 160 x 95 mm, 173 parts, among them J1 Display, J10 Analog CH1, J11 Analog CH2, J12 Analog CH3, J13 Analog CH4, J14 Analog CH5, J15 Micro_SD_Card, J16 OXY, J17 I2C, J18 SPI, J19 GPIO, J2 BIAS, J20 3V3, J21 GND, J22 5V, J3 SRB, J4 EEG Out, J5 Device Electrodes, J6 REF, J7 Analog CH6, J8 Analog CH7, J9 Analog CH0, Q1 BSH203,215, Q2 BSH203,215, Q3 BSH203,215, Q4 BSH203,215, Q5 BSH203,215, SW1 MAIN, U1 ESP32-DevKitC, U10 TLV840C, U11 PCF8574, U12 TSC2003, U2 ADS1299-x, U3 BHI160, U4 MCP3564RT, U5 LM1117-5.0, U6 NCV8165, U7 NCP115, U8 MIC5209, U9 NUF6401, X1 ECS-2520MVLC-020.48-BN-TR

Commit message: redesigned board partially
Parts:
- moved J1 47.3 mm to (41.2, 43.2), turned to -90 degrees
- moved J19 37.4 mm to (65.5, 41.8), turned to 180 degrees
- moved TP10 36.4 mm to (43.2, 48.5)
- moved TP11 31.5 mm to (45.5, 47.1)
- moved TP9 26.7 mm to (48.7, 46.0)
- moved JP11 23.1 mm to (55.8, 58.0), turned to 0 degrees
- moved JP12 23.0 mm to (52.1, 55.4), turned to 0 degrees
- moved C46 19.4 mm to (50.2, 43.1), turned to -90 degrees
- moved JP10 18.5 mm to (59.5, 56.1), turned to 90 degrees
- moved C47 17.6 mm to (51.5, 42.7), turned to -90 degrees
- moved J18 12.5 mm to (53.8, 4.10), turned to 90 degrees
- moved U11 10.8 mm to (57.4, 47.2), turned to 90 degrees
- moved U1 9.05 mm to (24.6, 24.3), turned to -90 degrees
- moved TP13 6.95 mm to (103.1, 63.5)
- moved JP9 5.02 mm to (51.4, 69.5)
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Routing:
- net +3V3: track 386.0 -> 60.0 mm, vias 12 -> 4
- net /VSPI_MOSI: track 276.0 -> 30.5 mm, vias 4 -> 3
- net /I2C1_SDA: track 256.4 -> 23.7 mm, vias 3 -> 2
- net /VSPI_SCK: track 277.7 -> 49.7 mm, vias 5 -> 3
- net /I2C1_SCK: track 249.3 -> 25.5 mm, vias 3 -> 2
- net /VSPI_MISO: track 273.7 -> 50.9 mm, vias 4 -> 3
- net +5V: track 198.7 -> 35.9 mm, vias 3 -> 0
- net /~{ADC_INT}: track 143.0 -> 0.00 mm, vias 1 -> 0
- net /3V3_SW: track 140.8 -> 8.87 mm, vias 14 -> 0
- net +6V: track 147.7 -> 27.5 mm, vias 5 -> 0
- net /ADC_CS: track 111.5 -> 0.00 mm, vias 1 -> 0
- net +3.3VA: track 76.5 -> 0.00 mm, vias 1 -> 0
- net /EKG/EEGMux/BIAS: track 69.0 -> 0.00 mm
- net /LCD_DC: track 12.6 -> 76.6 mm
- net /LCD_BL: track 18.4 -> 76.3 mm
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- removed copper zone on B.Cu, net AVSS
- removed copper zone on F.Cu, net AVSS
Other:
- rule pad_to_mask_clearance: 0 -> 0.05

Commit message: finished layout for review
Parts:
- removed H4: MountingHole, ownLib:MountingHole_3.2mm_M3_no_Mask
- removed TP27: DET_A, TestPoint:TestPoint_Pad_D1.0mm
- removed TP28: DET_B, TestPoint:TestPoint_Pad_D1.0mm
- added H3: MountingHole, ownLib:MountingHole_3.2mm_M3_no_Mask, F.Cu at (155.0, 90.0)
- U4: footprint Package_SO:HTSSOP-20-1EP_4.4x6.5mm_P0.65mm_EP3.4x6.5mm_Mask2.75x3.43mm -> ownLib:HTSSOP-20-1EP_4.4x6.5mm_P0.65mm_3.4x6.5mm_Mask2.75x3.43mm
- moved J18 42.8 mm to (96.6, 4.60)
- moved J17 27.1 mm to (84.3, 4.60)
- moved TP12 7.21 mm to (123.4, 14.6)
- moved JP1 6.88 mm to (138.1, 80.3)
- moved TP10 6.55 mm to (49.6, 47.1)
- moved C1 3.23 mm to (135.0, 87.6)
- moved R5 3.23 mm to (138.2, 85.6)
- moved R6 3.23 mm to (136.6, 87.6)
- moved TP9 1.56 mm to (47.6, 47.1)
- moved J15 1.34 mm to (9.29, 69.1)
- moved FB3 0.20 mm to (4.00, 61.1)
- moved C19 0.12 mm to (77.9, 53.3)
Connections:
- J15 pad 10: Net-(J15-Pad10) -> +3V3
- J15 pad 9: Net-(J15-Pad9) -> /CardDet
- J19 pad 2: /BreadBoard/P0 -> /CardDet
- U11 pad 4: /BreadBoard/P0 -> /CardDet
- U2 pad 27: Net-(U2-Pad27) -> unconnected-(U2-Pad27)
- U2 pad 29: Net-(U2-Pad27) -> unconnected-(U2-Pad29)
- U3 pad 1: Net-(U3-Pad1) -> unconnected-(U3-Pad1)
- U3 pad 14: Net-(U3-Pad1) -> unconnected-(U3-Pad14)
- U3 pad 15: Net-(U3-Pad1) -> unconnected-(U3-Pad15)
- U3 pad 16: Net-(U3-Pad1) -> unconnected-(U3-Pad16)
- U3 pad 17: Net-(U3-Pad1) -> unconnected-(U3-Pad17)
- U3 pad 19: Net-(U3-Pad1) -> unconnected-(U3-Pad19)
- U3 pad 2: Net-(U3-Pad1) -> unconnected-(U3-Pad2)
- U3 pad 22: Net-(U3-Pad1) -> unconnected-(U3-Pad22)
- U3 pad 4: Net-(U3-Pad1) -> unconnected-(U3-Pad4)
- U3 pad 5: Net-(U3-Pad1) -> unconnected-(U3-Pad5)
- U3 pad 6: Net-(U3-Pad1) -> unconnected-(U3-Pad6)
- U5 pad 4: (no net) -> +5V
- U6 pad 2: Net-(U6-Pad2) -> unconnected-(U6-Pad2)
- U6 pad 3: Net-(U6-Pad2) -> unconnected-(U6-Pad3)
- U6 pad 6: Net-(U6-Pad2) -> unconnected-(U6-Pad6)
- U6 pad 7: Net-(U6-Pad2) -> unconnected-(U6-Pad7)
Routing:
- net +3V3: track 60.0 -> 416.7 mm, vias 4 -> 7
- net /VSPI_MOSI: track 30.5 -> 331.0 mm, vias 3 -> 4
- net /VSPI_SCK: track 49.7 -> 348.3 mm, vias 3 -> 7
- net /VSPI_MISO: track 50.9 -> 341.3 mm, vias 3 -> 4
- net /3V3_SW: track 8.87 -> 218.0 mm, vias 0 -> 9
- net /I2C1_SCK: track 25.5 -> 224.7 mm, vias 2 -> 4
- net /I2C1_SDA: track 23.7 -> 219.2 mm, vias 2 -> 4
- net +5V: track 35.9 -> 228.5 mm, vias 0 -> 2
- net /SIG_SW: track 0.00 -> 172.2 mm, vias 0 -> 6
- net /ADC_CS: track 0.00 -> 154.3 mm
- net +6V: track 27.5 -> 172.9 mm, vias 0 -> 3
- net /~{EKG_INT}: track 10.3 -> 130.7 mm
- net /~{ADC_INT}: track 0.00 -> 118.0 mm, vias 0 -> 1
- net /~{SDPowerOK}: track 10.6 -> 117.5 mm, vias 0 -> 2
- net /~{SDPowerUp}: track 2.01 -> 105.9 mm, vias 0 -> 2
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- added copper zone on B.Cu, net AVSS
- added copper zone on F.Cu, net AVSS
Other:
- outline, holes or cut-outs redrawn
- board text added: "1P 1N 2P 2N 3P 3N 4P 4N BIAS"
- board text added: "3V3"
- board text added: "3V3|SCK|SDA|GND"
- board text added: "3V3|SIG|GND"
- board text added: "5V"
- board text added: "A0"
- board text added: "A1"
- board text added: "A2"
- board text added: "ADC"
- board text added: "ADC CS"
- board text added: "ASCK"
- board text added: "ASDA"
- board text added: "Addr"
- board text added: "Analog power supply"
- board text added: "BIAS Filter"
- board text added: "BIASINV"
- board text added: "BIASOUT"
- board text added: "Battery - | +"
- board text added: "CH0"
- board text added: "CH1"
- board text added: "CH2"
- board text added: "CH3"
- board text added: "CH4"
- board text added: "CH5"
- board text added: "CH6"
- board text added: "CH7"
- board text added: "COM"
- board text added: "COM 1P 2P 3P 4P BIAS"
- board text added: "Clock"
- board text added: "Display"
- board text added: "EKG"
- board text added: "EKG CS GPIO1 GPIO2 GPIO3 GPIO4"
- board text added: "EKG Default Configuration"
- board text added: "ESP32-DevKit-C4"
- board text added: "Filled = Set"
- board text added: "Filter"
- board text added: "Filter Out"
- board text added: "GND"
- board text added: "GND IO7 IO6 GND IO5 IO4 GND IO3 IO2 GND"
- board text added: "GND|SCK|MOSI|MISO|3V3"
- board text added: "GPIO Expander"
- board text added: "GPIO1"
- board text added: "GPIO2"
- board text added: "IMU"
- board text added: "IN1"
- board text added: "IN1N"
- board text added: "IN2"
- board text added: "IN2N"
- board text added: "IN3N"
- board text added: "IN4N"
- board text added: "IN|INV|OUT|REF|SEL"
- board text added: "IO1 IO0 GND"
- board text added: "MCK"
- board text added: "MISO"
- board text added: "MOSI"
- board text added: "OUT"
- board text added: "PU0"
- board text added: "PU1"
- board text added: "Power supply"
- board text added: "Pulsoxymeter"
- board text added: "PwrOK"
- board text added: "PwrUp"
- board text added: "REFIN- ----- REFIN+"
- board text added: "RES MISO SCK MOSI CS RES"
- board text added: "Routing to"
- board text added: "SCK"
- board text added: "SD Card"
- board text added: "SDA"
- board text added: "SRB"
- board text added: "SW"
- board text added: "Touch"
- board text added: "VSPI"
- board text added: "Vcc|SDA|SCK|GND"
- board text added: "Vsel"

Commit message: did some minor changes
Parts:
- added G***: LOGO, ownLib:LogoMate7x7, F.Cu at (16.4, 5.40)
- JP1: value BIASOUT SEL -> FILTER OUT
- moved J15 0.22 mm to (9.50, 69.2)
Routing:
- net /CardDet: track 103.8 -> 102.9 mm
- net AVSS: vias 926 -> 933
Other:
- board text added: "Designed by Patrick Hanner 2022 github.com/useless-branch"
- board text added: "x"
- board text added: "y"

Commit message: worked feedback into layout
Parts:
- added R27: 2k2, Resistor_SMD:R_0402_1005Metric, F.Cu at (75.9, 52.3)
- added R28: 2k2, Resistor_SMD:R_0402_1005Metric, F.Cu at (82.5, 47.5)
- added R29: 100k, Resistor_SMD:R_0402_1005Metric, F.Cu at (17.5, 69.9)
- moved G*** 97.4 mm to (98.9, 57.1)
- moved TP4 3.08 mm to (83.8, 47.0)
- moved TP3 1.90 mm to (74.1, 51.8)
Routing:
- net /3V3_SW: track 218.0 -> 223.7 mm
- net /IMU/ASDA: track 2.15 -> 4.97 mm
- net /IMU/ASCK: track 3.31 -> 5.25 mm
- net /CardDet: track 102.9 -> 104.6 mm
- net /LCD_RST: track 66.2 -> 67.2 mm
- net /~{SDPowerUp}: track 105.9 -> 106.8 mm
- net AVSS: vias 933 -> 977
Other:
- board text added: "A"
- board text added: "Designed by Patrick Hanner 2022 Resources available at: github.com/useless-branch"
- board text added: "EduSignal v1"
- board text added: "FAIL"
- board text added: "For educational and development purposes only!"
- board text added: "GND|SIG|3V3"
- board text added: "JLCJLCJLCJLC"
- board text added: "NOT FOR MEDICAL USE!"
- board text added: "OK"
- board text removed: "Designed by Patrick Hanner 2022 github.com/useless-branch"
