File: board/board.kicad_pcb (KiCad board)
At the start: 4 copper layers, 160 x 95 mm, 175 parts, among them J1 Display, J10 Analog CH1, J11 Analog CH2, J12 Analog CH3, J13 Analog CH4, J14 Analog CH5, J15 Micro_SD_Card, J16 OXY, J17 I2C, J18 SPI, J19 GPIO, J2 BIAS, J20 3V3, J21 GND, J22 5V, J3 SRB, J4 EEG Out, J5 Device Electrodes, J6 REF, J7 Analog CH6, J8 Analog CH7, J9 Analog CH0, Q1 BSH203,215, Q2 BSH203,215, Q3 BSH203,215, Q4 BSH203,215, Q5 BSH203,215, SW1 MAIN, U1 ESP32-DevKitC, U10 TLV840C, U11 PCF8574, U12 TSC2003, U2 ADS1299-x, U3 BHI160, U4 MCP3564RT, U5 LM1117-5.0, U6 NCV8165, U7 NCP115, U8 MIC5209, U9 NUF6401, X1 ECS-2520MVLC-020.48-BN-TR

Commit message: did some minor stuff
Parts:
- moved TP4 0.35 mm to (84.2, 47.0)
Routing:
- net /IMU/ASDA: track 4.97 -> 5.52 mm
- net /3V3_SW: track 223.7 -> 224.2 mm
- net AVSS: vias 977 -> 1009
Other:
- board text added: "AVSS -X -Y +X +Y BL RST DC CS MOSI MISO SCK 3V3 5V GND"
- board text added: "GND IO7 IO6 GND IO5 IO4 GND IO3 IO2 GND IO1 IO0 GND"
- board text removed: "GND IO7 IO6 GND IO5 IO4 GND IO3 IO2 GND"
- board text removed: "IO1 IO0 GND"

Commit message: worked feedback into layout with dp
Parts:
- added C51: 100n, Capacitor_SMD:C_0402_1005Metric, F.Cu at (140.1, 25.3)
- added C52: 100n, Capacitor_SMD:C_0402_1005Metric, F.Cu at (116.0, 80.7)
- added TP27: RX, TestPoint:TestPoint_Pad_D1.0mm, F.Cu at (54.1, 37.6)
- added TP28: TX, TestPoint:TestPoint_Pad_D1.0mm, F.Cu at (57.1, 37.6)
- moved R4 29.6 mm to (119.1, 44.6), turned to -90 degrees
- moved R3 16.9 mm to (117.3, 48.9), turned to 90 degrees
- moved C42 7.43 mm to (16.9, 61.5), turned to 90 degrees
- moved C43 6.98 mm to (15.1, 61.0)
- moved R8 2.38 mm to (115.3, 73.3), turned to 90 degrees
- moved C7 2.06 mm to (120.1, 74.8), turned to -90 degrees
- moved C12 1.70 mm to (118.1, 74.4), turned to 0 degrees
- moved C8 1.37 mm to (119.1, 76.6)
Connections:
- C11 pad 1: +3V3 -> +5VA
- U1 pad 23: unconnected-(U1-Pad23) -> Net-(TP28-Pad1)
- U1 pad 24: unconnected-(U1-Pad24) -> Net-(TP27-Pad1)
- U2 pad 19: +3V3 -> +5VA
- U2 pad 21: +3V3 -> +5VA
- U2 pad 22: +3V3 -> +5VA
- U2 pad 56: +3V3 -> +5VA
- U2 pad 59: +3V3 -> +5VA
Routing:
- net /MCLK: track 77.9 -> 4.97 mm
- net /ADC/MCLK: track 1.76 -> 40.4 mm
- net +6V: track 172.8 -> 209.8 mm
- net /EKG/MCLK: track 1.43 -> 35.8 mm
- net +5VA: track 41.3 -> 74.9 mm, vias 0 -> 2
- net +3V3: track 416.7 -> 390.5 mm, vias 7 -> 4
- net Net-(TP28-Pad1): track 0.00 -> 23.8 mm, vias 0 -> 2
- net Net-(TP27-Pad1): track 0.00 -> 23.2 mm, vias 0 -> 2
- net /CardDet: track 104.6 -> 92.1 mm
- net /ADC_CS: track 154.3 -> 164.9 mm
- net /IMU_INT: track 69.8 -> 78.2 mm
- net Net-(R8-Pad2): track 2.39 -> 5.17 mm
- net Net-(C39-Pad1): track 34.6 -> 31.9 mm
- net /~{EKG_INT}: track 130.3 -> 132.6 mm
- net +3.3VA: track 86.0 -> 87.1 mm
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Other:
- board text added: "RX|TX"

Commit message: updated gerber data
Routing:
- net AVSS: vias 1028 -> 1033
Changed lines of the file:
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@@
     (pad_to_mask_clearance 0.05)
     (pcbplotparams
-      (layerselection 0x0001030_ffffffff)
+      (layerselection 0x00010fc_ffffffff)
       (disableapertmacros false)
       (usegerberextensions false)
@@
       (sketchpadsonfab false)
       (subtractmaskfromsilk false)
-      (outputformat 4)
+      (outputformat 1)
       (mirror false)
-      (drillshape 2)
+      (drillshape 0)
       (scaleselection 1)
-      (outputdirectory "pdf")
+      (outputdirectory "gbr")
     )
   )
@@
     )
     (fp_line (start -7 -6.25) (end -6 -6.25) (layer "F.SilkS") (width 0.12))
-    (fp_line (start -7 -6.25) (end -7 6.25) (layer "F.SilkS") (width 0.12))
     (fp_line (start 7 -6.25) (end 7 7.25) (layer "F.SilkS") (width 0.12))
-    (fp_line (start -3.75 -6.25) (end -0.5 -6.25) (layer "F.SilkS") (width 0.12))
+    (fp_line (start 5.5 8.75) (end 2.5 8.75) (layer "F.SilkS") (width 0.12))
+    (fp_line (start -7 -6.25) (end -7 6.25) (layer "F.SilkS") (width 0.12))
     (fp_line (start 2 -6.25) (end 7 -6.25) (layer "F.SilkS") (width 0.12))
     (fp_line (start 2.5 8.75) (end 2.5 5.75) (layer "F.SilkS") (width 0.12))
-    (fp_line (start 5.5 8.75) (end 2.5 8.75) (layer "F.SilkS") (width 0.12))
+    (fp_line (start -3.75 -6.25) (end -0.5 -6.25) (layer "F.SilkS") (width 0.12))
     (fp_rect (start -7.5 -6.75) (end 7.5 9.75) (layer "F.CrtYd") (width 0.05) (fill none))
     (pad "1" smd roundrect (at 1.94 4.75 270) (size 0.8 2) (layers "F.Cu" "F.Paste" "F.Mask") (roundrect_rratio 0.25)
@@
     (pad "10" smd roundrect (at -4.95 -5.85 270) (size 1.8 1.4) (layers "F.Cu" "F.Paste" "F.Mask") (roundrect_rratio 0.25)
       (net 10 "+3V3") (pinfunction "DET_A") (pintype "passive"))
-    (pad "11" smd roundrect (at 6.6 8.3 270) (size 1.4 1.9) (layers "F.Cu" "F.Paste" "F.Mask") (roundrect_rratio 0.25)
-      (net 37 "Net-(FB3-Pad1)") (pinfunction "SHIELD") (pintype "passive"))
     (pad "11" smd roundrect (at -6.55 7.3 270) (size 1.4 1.9) (layers "F.Cu" "F.Paste" "F.Mask") (roundrect_rratio 0.25)
       (net 37 "Net-(FB3-Pad1)") (pinfunction "SHIELD") (pintype "passive"))
+    (pad "11" smd roundrect (at 6.6 8.3 270) (size 1.4 1.9) (layers "F.Cu" "F.Paste" "F.Mask") (roundrect_rratio 0.25)
+      (net 37 "Net-(FB3-Pad1)") (pinfunction "SHIELD") (pintype "passive"))
     (zone (net 0) (net_name "") (layers *.Cu) (name "KEEP OUT") (hatch edge 0.508)
       (connect_pads (clearance 0))
       (min_thickness 0.254)
-      (keepout (tracks not_allowed) (vias not_allowed) (pads not_allowed ) (copperpour not_allowed) (footprints not_allowed))
+      (keepout (tracks not_allowed) (vias allowed) (pads not_allowed ) (copperpour not_allowed) (footprints not_allowed))
       (fill (thermal_gap 0.508) (thermal_bridge_width 0.508))
       (polygon
@@
   (via (at 117.55 64.45) (size 0.45) (drill 0.2) (layers "F.Cu" "B.Cu") (free) (net 2))
   (via (at 106 68) (size 0.45) (drill 0.2) (layers "F.Cu" "B.Cu") (free) (net 2))
+  (via (at 10.9 66.2) (size 0.45) (drill 0.2) (layers "F.Cu" "B.Cu") (free) (net 2))
   (via (at 153 11.25) (size 0.6) (drill 0.3) (layers "F.Cu" "B.Cu") (free) (net 2))
   (via (at 5 52.5) (size 0.45) (drill 0.2) (layers "F.Cu" "B.Cu") (free) (net 2))
@@
   (via (at 46 38.2) (size 0.45) (drill 0.2) (layers "F.Cu" "B.Cu") (free) (net 2))
   (via (at 128.25 23) (size 0.45) (drill 0.2) (layers "F.Cu" "B.Cu") (free) (net 2))
+  (via (at 9.3 66.8) (size 0.45) (drill 0.2) (layers "F.Cu" "B.Cu") (free) (net 2))
   (via (at 90 80.25) (size 0.6) (drill 0.3) (layers "F.Cu" "B.Cu") (free) (net 2))
   (via (at 143 22.25) (size 0.45) (drill 0.2) (layers "F.Cu" "B.Cu") (free) (net 2))
@@
   (via (at 5.85 49) (size 0.45) (drill 0.2) (layers "F.Cu" "B.Cu") (free) (net 2))
   (via (at 41.066565 36.461308) (size 0.45) (drill 0.2) (layers "F.Cu" "B.Cu") (free) (net 2))
+  (via (at 12.6 61.9) (size 0.45) (drill 0.2) (layers "F.Cu" "B.Cu") (free) (net 2))
   (via (at 106.1 83.4) (size 0.45) (drill 0.2) (layers "F.Cu" "B.Cu") (free) (net 2))
   (via (at 6.1 55.2) (size 0.45) (drill 0.2) (layers "F.Cu" "B.Cu") (free) (net 2))
@@
   (via (at 10 19.25) (size 0.6) (drill 0.3) (layers "F.Cu" "B.Cu") (free) (net 2))
   (via (at 84.5 71.25) (size 0.6) (drill 0.3) (layers "F.Cu" "B.Cu") (free) (net 2))
+  (via (at 13.5 72.2) (size 0.45) (drill 0.2) (layers "F.Cu" "B.Cu") (free) (net 2))
   (via (at 61.8 65.6) (size 0.45) (drill 0.2) (layers "F.Cu" "B.Cu") (free) (net 2))
   (via (at 13.7 61.6) (size 0.45) (drill 0.2) (layers "F.Cu" "B.Cu") (free) (net 2))
@@
   (via (at 143.25 30.5) (size 0.6) (drill 0.3) (layers "F.Cu" "B.Cu") (free) (net 2))
   (via (at 61.4 46.825) (size 0.45) (drill 0.2) (layers "F.Cu" "B.Cu") (free) (net 2))
+  (via (at 10.9 71.3) (size 0.45) (drill 0.2) (layers "F.Cu" "B.Cu") (free) (net 2))
   (via (at 159 42) (size 0.45) (drill 0.2) (layers "F.Cu" "B.Cu") (free) (net 2))
   (via (at 116.5 94) (size 0.45) (drill 0.2) (layers "F.Cu" "B.Cu") (free) (net 2))
