File: board/imu.kicad_sch (KiCad schematic)
At the start: 6 parts

Commit message: updated hw project
Parts:
- C?: value (none) -> 470n
- C? (x2): value (none) -> 100n
- C?: value (none) -> 1u
- JP?: value (none) -> AddrSelect
- U?: value (none) -> BHI160
Changed lines of the file:
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@@
     (in_bom yes) (on_board yes) (fields_autoplaced)
     (property "Reference" "U?" (id 0) (at 158.75 69.85 0))
-    (property "Value" "" (id 1) (at 158.75 72.39 0))
+    (property "Value" "BHI160" (id 1) (at 158.75 72.39 0))
     (property "Footprint" "" (id 2) (at 207.01 83.82 0)
       (effects (font (size 1.27 1.27)) hide)
@@
       (effects (font (size 1.27 1.27)) hide)
     )
-    (property "Value" "" (id 1) (at 119.38 72.39 0))
+    (property "Value" "VDDA" (id 1) (at 119.38 72.39 0))
     (property "Footprint" "" (id 2) (at 119.38 77.47 0)
       (effects (font (size 1.27 1.27)) hide)
@@
       (effects (font (size 1.27 1.27)) hide)
     )
-    (property "Value" "" (id 1) (at 124.46 80.0099 90)
+    (property "Value" "VDD" (id 1) (at 124.46 80.0099 90)
       (effects (font (size 1.27 1.27)) (justify left))
     )
@@
       (effects (font (size 1.27 1.27)) (justify left))
     )
-    (property "Value" "" (id 1) (at 139.7 93.9862 0)
+    (property "Value" "470n" (id 1) (at 139.7 93.9862 0)
       (effects (font (size 1.27 1.27)) (justify left))
     )
@@
       (effects (font (size 1.27 1.27)) (justify left))
     )
-    (property "Value" "" (id 1) (at 121.92 90.1762 0)
+    (property "Value" "100n" (id 1) (at 121.92 90.1762 0)
       (effects (font (size 1.27 1.27)) (justify left))
     )
@@
       (effects (font (size 1.27 1.27)) (justify left))
     )
-    (property "Value" "" (id 1) (at 130.81 85.0962 0)
+    (property "Value" "1u" (id 1) (at 130.81 85.0962 0)
       (effects (font (size 1.27 1.27)) (justify left))
     )
@@
       (effects (font (size 1.27 1.27)) hide)
     )
-    (property "Value" "" (id 1) (at 104.14 90.17 0))
+    (property "Value" "VDD" (id 1) (at 104.14 90.17 0))
     (property "Footprint" "" (id 2) (at 104.14 95.25 0)
       (effects (font (size 1.27 1.27)) hide)
@@
       (effects (font (size 1.27 1.27)) (justify left))
     )
-    (property "Value" "" (id 1) (at 139.7 85.0962 0)
+    (property "Value" "100n" (id 1) (at 139.7 85.0962 0)
       (effects (font (size 1.27 1.27)) (justify left))
     )
@@
       (effects (font (size 1.27 1.27)) (justify left))
     )
-    (property "Value" "" (id 1) (at 101.6 102.8699 90)
+    (property "Value" "AddrSelect" (id 1) (at 101.6 102.8699 90)
       (effects (font (size 1.27 1.27)) (justify left))
     )
@@
       (effects (font (size 1.27 1.27)) hide)
     )
-    (property "Value" "" (id 1) (at 115.57 96.52 0))
+    (property "Value" "GND" (id 1) (at 115.57 96.52 0))
     (property "Footprint" "" (id 2) (at 119.38 96.52 0)
       (effects (font (size 1.27 1.27)) hide)
@@
       (effects (font (size 1.27 1.27)) hide)
     )
-    (property "Value" "" (id 1) (at 104.14 113.03 0))
+    (property "Value" "GND" (id 1) (at 104.14 113.03 0))
     (property "Footprint" "" (id 2) (at 104.14 107.95 0)
       (effects (font (size 1.27 1.27)) hide)

Commit message: updated schematic
Connections:
- net VDD renamed +3V3
- net VDDA renamed +3.3VA
Changed lines of the file:
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@@
   (junction (at 137.16 86.36) (diameter 0) (color 0 0 0 0)
   )
+  (junction (at 137.16 96.52) (diameter 0) (color 0 0 0 0)
+  )
+  (junction (at 119.38 96.52) (diameter 0) (color 0 0 0 0)
+  )
+  (junction (at 119.38 77.47) (diameter 0) (color 0 0 0 0)
+  )
   (junction (at 128.27 80.01) (diameter 0) (color 0 0 0 0)
-  )
-  (junction (at 137.16 96.52) (diameter 0) (color 0 0 0 0)
-  )
-  (junction (at 119.38 96.52) (diameter 0) (color 0 0 0 0)
-  )
-  (junction (at 119.38 77.47) (diameter 0) (color 0 0 0 0)
   )
   (junction (at 128.27 96.52) (diameter 0) (color 0 0 0 0)
@@
   (hierarchical_label "INT" (shape output) (at 147.32 109.22 180)
     (effects (font (size 1.27 1.27)) (justify right))
+  )
+  (symbol (lib_id "power:+3V3") (at 128.27 80.01 90) (unit 1)
+    (in_bom yes) (on_board yes) (fields_autoplaced)
+    (property "Reference" "#PWR?" (id 0) (at 132.08 80.01 0)
+      (effects (font (size 1.27 1.27)) hide)
+    )
+    (property "Value" "+3V3" (id 1) (at 124.46 80.0099 90)
+      (effects (font (size 1.27 1.27)) (justify left))
+    )
+    (property "Footprint" "" (id 2) (at 128.27 80.01 0)
+      (effects (font (size 1.27 1.27)) hide)
+    )
+    (property "Datasheet" "" (id 3) (at 128.27 80.01 0)
+      (effects (font (size 1.27 1.27)) hide)
+    )
+    (pin "1")
   )
   (symbol (lib_id "ownLib:BHI160") (at 172.72 66.04 0) (unit 1)
@@
       (effects (font (size 1.27 1.27)) hide)
     )
-    (property "Datasheet" "" (id 3) (at 207.01 83.82 0)
+    (property "Datasheet" "https://www.mouser.de/pdfdocs/Bosch-BST-BHI160B-DS000-01-Datasheet.pdf" (id 3) (at 207.01 83.82 0)
       (effects (font (size 1.27 1.27)) hide)
     )
@@
     (pin "9")
   )
-  (symbol (lib_id "power:VDDA") (at 119.38 77.47 0) (unit 1)
+  (symbol (lib_id "Device:C_Small") (at 137.16 92.71 0) (unit 1)
+    (in_bom yes) (on_board yes) (fields_autoplaced)
+    (property "Reference" "C?" (id 0) (at 139.7 91.4462 0)
+      (effects (font (size 1.27 1.27)) (justify left))
+    )
+    (property "Value" "470n" (id 1) (at 139.7 93.9862 0)
+      (effects (font (size 1.27 1.27)) (justify left))
+    )
+    (property "Footprint" "" (id 2) (at 137.16 92.71 0)
+      (effects (font (size 1.27 1.27)) hide)
+    )
+    (property "Datasheet" "~" (id 3) (at 137.16 92.71 0)
+      (effects (font (size 1.27 1.27)) hide)
+    )
+    (pin "1")
+    (pin "2")
+  )
+  (symbol (lib_id "Device:C_Small") (at 119.38 88.9 0) (unit 1)
+    (in_bom yes) (on_board yes) (fields_autoplaced)
+    (property "Reference" "C?" (id 0) (at 121.92 87.6362 0)
+      (effects (font (size 1.27 1.27)) (justify left))
+    )
+    (property "Value" "100n" (id 1) (at 121.92 90.1762 0)
+      (effects (font (size 1.27 1.27)) (justify left))
+    )
+    (property "Footprint" "" (id 2) (at 119.38 88.9 0)
+      (effects (font (size 1.27 1.27)) hide)
+    )
+    (property "Datasheet" "~" (id 3) (at 119.38 88.9 0)
+      (effects (font (size 1.27 1.27)) hide)
+    )
+    (pin "1")
+    (pin "2")
+  )
+  (symbol (lib_id "power:+3.3VA") (at 119.38 77.47 0) (unit 1)
     (in_bom yes) (on_board yes) (fields_autoplaced)
     (property "Reference" "#PWR?" (id 0) (at 119.38 81.28 0)
       (effects (font (size 1.27 1.27)) hide)
     )
-    (property "Value" "VDDA" (id 1) (at 119.38 72.39 0))
+    (property "Value" "+3.3VA" (id 1) (at 119.38 72.39 0))
     (property "Footprint" "" (id 2) (at 119.38 77.47 0)
       (effects (font (size 1.27 1.27)) hide)
@@
     (pin "1")
   )
-  (symbol (lib_id "power:VDD") (at 128.27 80.01 90) (unit 1)
-    (in_bom yes) (on_board yes) (fields_autoplaced)
-    (property "Reference" "#PWR?" (id 0) (at 132.08 80.01 0)
-      (effects (font (size 1.27 1.27)) hide)
-    )
-    (property "Value" "VDD" (id 1) (at 124.46 80.0099 90)
-      (effects (font (size 1.27 1.27)) (justify left))
-    )
-    (property "Footprint" "" (id 2) (at 128.27 80.01 0)
-      (effects (font (size 1.27 1.27)) hide)
-    )
-    (property "Datasheet" "" (id 3) (at 128.27 80.01 0)
-      (effects (font (size 1.27 1.27)) hide)
-    )
-    (pin "1")
-  )
-  (symbol (lib_id "Device:C_Small") (at 137.16 92.71 0) (unit 1)
-    (in_bom yes) (on_board yes) (fields_autoplaced)
-    (property "Reference" "C?" (id 0) (at 139.7 91.4462 0)
-      (effects (font (size 1.27 1.27)) (justify left))
-    )
-    (property "Value" "470n" (id 1) (at 139.7 93.9862 0)
-      (effects (font (size 1.27 1.27)) (justify left))
-    )
-    (property "Footprint" "" (id 2) (at 137.16 92.71 0)
-      (effects (font (size 1.27 1.27)) hide)
-    )
-    (property "Datasheet" "~" (id 3) (at 137.16 92.71 0)
-      (effects (font (size 1.27 1.27)) hide)
-    )
-    (pin "1")
-    (pin "2")
-  )
-  (symbol (lib_id "Device:C_Small") (at 119.38 88.9 0) (unit 1)
-    (in_bom yes) (on_board yes) (fields_autoplaced)
-    (property "Reference" "C?" (id 0) (at 121.92 87.6362 0)
-      (effects (font (size 1.27 1.27)) (justify left))
-    )
-    (property "Value" "100n" (id 1) (at 121.92 90.1762 0)
-      (effects (font (size 1.27 1.27)) (justify left))
-    )
-    (property "Footprint" "" (id 2) (at 119.38 88.9 0)
-      (effects (font (size 1.27 1.27)) hide)
-    )
-    (property "Datasheet" "~" (id 3) (at 119.38 88.9 0)
-      (effects (font (size 1.27 1.27)) hide)
-    )
-    (pin "1")
-    (pin "2")
-  )
   (symbol (lib_id "Device:C_Small") (at 128.27 83.82 0) (unit 1)
     (in_bom yes) (on_board yes) (fields_autoplaced)
@@
     (pin "1")
     (pin "2")
-  )
-  (symbol (lib_id "power:VDD") (at 104.14 95.25 0) (unit 1)
-    (in_bom yes) (on_board yes) (fields_autoplaced)
-    (property "Reference" "#PWR?" (id 0) (at 104.14 99.06 0)
-      (effects (font (size 1.27 1.27)) hide)
-    )
-    (property "Value" "VDD" (id 1) (at 104.14 90.17 0))
-    (property "Footprint" "" (id 2) (at 104.14 95.25 0)
-      (effects (font (size 1.27 1.27)) hide)
-    )
-    (property "Datasheet" "" (id 3) (at 104.14 95.25 0)
-      (effects (font (size 1.27 1.27)) hide)
-    )
-    (pin "1")
   )
   (symbol (lib_id "Device:C_Small") (at 137.16 83.82 0) (unit 1)
@@
       (effects (font (size 1.27 1.27)) hide)
     )
+    (pin "1")
+  )
+  (symbol (lib_id "power:+3V3") (at 104.14 95.25 0) (unit 1)
+    (in_bom yes) (on_board yes) (fields_autoplaced)
+    (property "Reference" "#PWR?" (id 0) (at 104.14 99.06 0)
+      (effects (font (size 1.27 1.27)) hide)
+    )
+    (property "Value" "+3V3" (id 1) (at 106.68 93.9799 0)
+      (effects (font (size 1.27 1.27)) (justify left))
+    )
+    (property "Footprint" "" (id 2) (at 104.14 95.25 0)
+      (effects (font (size 1.27 1.27)) hide)
+    )
+    (property "Datasheet" "" (id 3) (at 104.14 95.25 0)
+      (effects (font (size 1.27 1.27)) hide)
+    )

Commit message: updated schematic
Connections:
- net +3.3VA renamed 3V3
Changed lines of the file:
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@@
   (junction (at 119.38 96.52) (diameter 0) (color 0 0 0 0)
-  )
-  (junction (at 119.38 77.47) (diameter 0) (color 0 0 0 0)
   )
   (junction (at 128.27 80.01) (diameter 0) (color 0 0 0 0)
@@
   (text "Low:  Address 0x28 (default)\nHigh: Address 0x29" (at 107.95 107.95 0)
     (effects (font (size 1.27 1.27)) (justify left bottom))
+  )
+  (hierarchical_label "3V3" (shape input) (at 119.38 77.47 180)
+    (effects (font (size 1.27 1.27)) (justify right))
   )
   (hierarchical_label "GPIO1" (shape bidirectional) (at 170.18 80.01 0)
@@
     (pin "2")
   )
-  (symbol (lib_id "power:+3.3VA") (at 119.38 77.47 0) (unit 1)
-    (in_bom yes) (on_board yes) (fields_autoplaced)
-    (property "Reference" "#PWR?" (id 0) (at 119.38 81.28 0)
-      (effects (font (size 1.27 1.27)) hide)
-    )
-    (property "Value" "+3.3VA" (id 1) (at 119.38 72.39 0))
-    (property "Footprint" "" (id 2) (at 119.38 77.47 0)
-      (effects (font (size 1.27 1.27)) hide)
-    )
-    (property "Datasheet" "" (id 3) (at 119.38 77.47 0)
-      (effects (font (size 1.27 1.27)) hide)
-    )
-    (pin "1")
-  )
   (symbol (lib_id "Device:C_Small") (at 128.27 83.82 0) (unit 1)

Commit message: ERC run
Parts:
- gave numbers to parts that had none: 6
Changed lines of the file:
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@@
   (symbol (lib_id "power:+3V3") (at 128.27 80.01 90) (unit 1)
     (in_bom yes) (on_board yes) (fields_autoplaced)
-    (property "Reference" "#PWR?" (id 0) (at 132.08 80.01 0)
+    (property "Reference" "#PWR019" (id 0) (at 132.08 80.01 0)
       (effects (font (size 1.27 1.27)) hide)
     )
@@
   (symbol (lib_id "ownLib:BHI160") (at 172.72 66.04 0) (unit 1)
     (in_bom yes) (on_board yes) (fields_autoplaced)
-    (property "Reference" "U?" (id 0) (at 158.75 69.85 0))
+    (property "Reference" "U3" (id 0) (at 158.75 69.85 0))
     (property "Value" "BHI160" (id 1) (at 158.75 72.39 0))
     (property "Footprint" "" (id 2) (at 207.01 83.82 0)
@@
   (symbol (lib_id "Device:C_Small") (at 137.16 92.71 0) (unit 1)
     (in_bom yes) (on_board yes) (fields_autoplaced)
-    (property "Reference" "C?" (id 0) (at 139.7 91.4462 0)
+    (property "Reference" "C21" (id 0) (at 139.7 91.4462 0)
       (effects (font (size 1.27 1.27)) (justify left))
     )
@@
   (symbol (lib_id "Device:C_Small") (at 119.38 88.9 0) (unit 1)
     (in_bom yes) (on_board yes) (fields_autoplaced)
-    (property "Reference" "C?" (id 0) (at 121.92 87.6362 0)
+    (property "Reference" "C18" (id 0) (at 121.92 87.6362 0)
       (effects (font (size 1.27 1.27)) (justify left))
     )
@@
   (symbol (lib_id "Device:C_Small") (at 128.27 83.82 0) (unit 1)
     (in_bom yes) (on_board yes) (fields_autoplaced)
-    (property "Reference" "C?" (id 0) (at 130.81 82.5562 0)
+    (property "Reference" "C19" (id 0) (at 130.81 82.5562 0)
       (effects (font (size 1.27 1.27)) (justify left))
     )
@@
   (symbol (lib_id "Device:C_Small") (at 137.16 83.82 0) (unit 1)
     (in_bom yes) (on_board yes) (fields_autoplaced)
-    (property "Reference" "C?" (id 0) (at 139.7 82.5562 0)
+    (property "Reference" "C20" (id 0) (at 139.7 82.5562 0)
       (effects (font (size 1.27 1.27)) (justify left))
     )
@@
   (symbol (lib_id "Jumper:Jumper_3_Bridged12") (at 104.14 101.6 90) (unit 1)
     (in_bom yes) (on_board yes) (fields_autoplaced)
-    (property "Reference" "JP?" (id 0) (at 101.6 100.3299 90)
+    (property "Reference" "JP8" (id 0) (at 101.6 100.3299 90)
       (effects (font (size 1.27 1.27)) (justify left))
     )
@@
   (symbol (lib_id "power:GND") (at 119.38 96.52 0) (unit 1)
     (in_bom yes) (on_board yes)
-    (property "Reference" "#PWR?" (id 0) (at 119.38 102.87 0)
+    (property "Reference" "#PWR018" (id 0) (at 119.38 102.87 0)
       (effects (font (size 1.27 1.27)) hide)
     )
@@
   (symbol (lib_id "power:+3V3") (at 104.14 95.25 0) (unit 1)
     (in_bom yes) (on_board yes) (fields_autoplaced)
-    (property "Reference" "#PWR?" (id 0) (at 104.14 99.06 0)
+    (property "Reference" "#PWR016" (id 0) (at 104.14 99.06 0)
       (effects (font (size 1.27 1.27)) hide)
     )
@@
   (symbol (lib_id "power:GND") (at 104.14 107.95 0) (unit 1)
     (in_bom yes) (on_board yes) (fields_autoplaced)
-    (property "Reference" "#PWR?" (id 0) (at 104.14 114.3 0)
+    (property "Reference" "#PWR017" (id 0) (at 104.14 114.3 0)
       (effects (font (size 1.27 1.27)) hide)
     )

Commit message: updated schematic after review
Other:
- note added: "Keep layout recommendation in mind"
- note added: "TODO: Pullup for AI2C"
Changed lines of the file:
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@@
     (stroke (width 0) (type default) (color 0 0 0 0))
+  )
+  (text "TODO: Pullup for AI2C" (at 177.8 92.71 0)
+    (effects (font (size 1.27 1.27)) (justify left bottom))
+  )
+  (text "Keep layout recommendation in mind\n" (at 137.16 66.04 0)
+    (effects (font (size 1.27 1.27)) (justify left bottom))
   )
   (text "Low:  Address 0x28 (default)\nHigh: Address 0x29" (at 107.95 107.95 0)

Commit message: added footprints to symbols and started layout
Parts:
- C18, C20, C21: footprint (none) -> Capacitor_SMD:C_0402_1005Metric
- C19: footprint (none) -> Capacitor_SMD:C_0603_1608Metric
- JP8: footprint (none) -> Jumper:SolderJumper-3_P1.3mm_Bridged12_Pad1.0x1.5mm
- U3: footprint (none) -> ownLib:BHI160
Changed lines of the file:
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@@
     (property "Reference" "U3" (id 0) (at 158.75 69.85 0))
     (property "Value" "BHI160" (id 1) (at 158.75 72.39 0))
-    (property "Footprint" "" (id 2) (at 207.01 83.82 0)
+    (property "Footprint" "ownLib:BHI160" (id 2) (at 207.01 83.82 0)
       (effects (font (size 1.27 1.27)) hide)
     )
@@
       (effects (font (size 1.27 1.27)) (justify left))
     )
-    (property "Footprint" "" (id 2) (at 137.16 92.71 0)
+    (property "Footprint" "Capacitor_SMD:C_0402_1005Metric" (id 2) (at 137.16 92.71 0)
       (effects (font (size 1.27 1.27)) hide)
     )
@@
       (effects (font (size 1.27 1.27)) (justify left))
     )
-    (property "Footprint" "" (id 2) (at 119.38 88.9 0)
+    (property "Footprint" "Capacitor_SMD:C_0402_1005Metric" (id 2) (at 119.38 88.9 0)
       (effects (font (size 1.27 1.27)) hide)
     )
@@
       (effects (font (size 1.27 1.27)) (justify left))
     )
-    (property "Footprint" "" (id 2) (at 128.27 83.82 0)
+    (property "Footprint" "Capacitor_SMD:C_0603_1608Metric" (id 2) (at 128.27 83.82 0)
       (effects (font (size 1.27 1.27)) hide)
     )
@@
       (effects (font (size 1.27 1.27)) (justify left))
     )
-    (property "Footprint" "" (id 2) (at 137.16 83.82 0)
+    (property "Footprint" "Capacitor_SMD:C_0402_1005Metric" (id 2) (at 137.16 83.82 0)
       (effects (font (size 1.27 1.27)) hide)
     )
@@
       (effects (font (size 1.27 1.27)) (justify left))
     )
-    (property "Footprint" "" (id 2) (at 104.14 101.6 0)
+    (property "Footprint" "Jumper:SolderJumper-3_P1.3mm_Bridged12_Pad1.0x1.5mm" (id 2) (at 104.14 101.6 0)
       (effects (font (size 1.27 1.27)) hide)
     )

Commit message: WIP pushed for meeting
Connections:
- net +3V3 is gone; now on net 3V3: C19.1, C20.1, JP8.3 (B), U3.8 (VDDIO)
Changed lines of the file:
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@@
   (junction (at 119.38 96.52) (diameter 0) (color 0 0 0 0)
-  )
-  (junction (at 128.27 80.01) (diameter 0) (color 0 0 0 0)
   )
   (junction (at 128.27 96.52) (diameter 0) (color 0 0 0 0)
@@
     (effects (font (size 1.27 1.27)) (justify left))
   )
+  (hierarchical_label "3V3" (shape input) (at 128.27 80.01 180)
+    (effects (font (size 1.27 1.27)) (justify right))
+  )
   (hierarchical_label "GPIO2" (shape bidirectional) (at 170.18 77.47 0)
     (effects (font (size 1.27 1.27)) (justify left))
   )
+  (hierarchical_label "3V3" (shape input) (at 104.14 95.25 90)
+    (effects (font (size 1.27 1.27)) (justify left))
+  )
   (hierarchical_label "SCK" (shape input) (at 147.32 104.14 180)
     (effects (font (size 1.27 1.27)) (justify right))
@@
   (hierarchical_label "INT" (shape output) (at 147.32 109.22 180)
     (effects (font (size 1.27 1.27)) (justify right))
-  )
-  (symbol (lib_id "power:+3V3") (at 128.27 80.01 90) (unit 1)
-    (in_bom yes) (on_board yes) (fields_autoplaced)
-    (property "Reference" "#PWR019" (id 0) (at 132.08 80.01 0)
-      (effects (font (size 1.27 1.27)) hide)
-    )
-    (property "Value" "+3V3" (id 1) (at 124.46 80.0099 90)
-      (effects (font (size 1.27 1.27)) (justify left))
-    )
-    (property "Footprint" "" (id 2) (at 128.27 80.01 0)
-      (effects (font (size 1.27 1.27)) hide)
-    )
-    (property "Datasheet" "" (id 3) (at 128.27 80.01 0)
-      (effects (font (size 1.27 1.27)) hide)
-    )
-    (pin "1")
   )
   (symbol (lib_id "ownLib:BHI160") (at 172.72 66.04 0) (unit 1)
@@
       (effects (font (size 1.27 1.27)) hide)
     )
-    (pin "1")
-  )
-  (symbol (lib_id "power:+3V3") (at 104.14 95.25 0) (unit 1)
-    (in_bom yes) (on_board yes) (fields_autoplaced)
-    (property "Reference" "#PWR016" (id 0) (at 104.14 99.06 0)
-      (effects (font (size 1.27 1.27)) hide)
-    )
-    (property "Value" "+3V3" (id 1) (at 106.68 93.9799 0)
-      (effects (font (size 1.27 1.27)) (justify left))
-    )
-    (property "Footprint" "" (id 2) (at 104.14 95.25 0)
-      (effects (font (size 1.27 1.27)) hide)
-    )
-    (property "Datasheet" "" (id 3) (at 104.14 95.25 0)
-      (effects (font (size 1.27 1.27)) hide)
-    )

Commit message: finished layout for review
Connections:
- now unconnected: U3.1, U3.14, U3.15, U3.16, U3.17, U3.19, U3.2, U3.22 (RESV4), U3.4 (RESV2), U3.5 (RESV3), U3.6
