File: board/imu.kicad_sch (KiCad schematic)
At the start: 6 parts, among them U3 BHI160

Commit message: worked feedback into layout
Other:
- note removed: "TODO: Pullup for AI2C"
Changed lines of the file:
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@@
     (stroke (width 0) (type default) (color 0 0 0 0))
-  )
-  (text "TODO: Pullup for AI2C" (at 177.8 92.71 0)
-    (effects (font (size 1.27 1.27)) (justify left bottom))
   )
   (text "Keep layout recommendation in mind\n" (at 137.16 66.04 0)

Commit message: did some minor stuff
Other:
- company: (none) -> Hochschule Pforzheim
- title: (none) -> eduSignal
Changed lines of the file:
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@@
 (kicad_sch (version 20211123) (generator eeschema)
   (paper "A4")
+  (title_block
+    (title "eduSignal")
+    (date "2022-07-14")
+    (rev "1")
+    (company "Hochschule Pforzheim")
+    (comment 1 "Patrick Hanner")
+    (comment 2 "Biosignal development board")
+  )
   (junction (at 128.27 86.36) (diameter 0) (color 0 0 0 0)
   )
