File: board/breadboard.kicad_sch (KiCad schematic)
At the start: 6 parts, among them J17 I2C, J18 SPI, J19 GPIO, J20 3V3, J21 GND, J22 5V

Commit message: added footprints to symbols and started layout
Parts:
- J17: footprint (none) -> Connector_PinHeader_2.54mm:PinHeader_1x04_P2.54mm_Vertical
- J18, J20, J21, J22: footprint (none) -> Connector_PinHeader_2.54mm:PinHeader_1x05_P2.54mm_Vertical
- J19: footprint (none) -> Connector_PinHeader_2.54mm:PinHeader_1x13_P2.54mm_Vertical
Changed lines of the file:
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@@
     (property "Reference" "J17" (id 0) (at 116.84 81.28 0))
     (property "Value" "I2C" (id 1) (at 116.84 83.82 0))
-    (property "Footprint" "" (id 2) (at 116.84 92.71 0)
+    (property "Footprint" "Connector_PinHeader_2.54mm:PinHeader_1x04_P2.54mm_Vertical" (id 2) (at 116.84 92.71 0)
       (effects (font (size 1.27 1.27)) hide)
     )
@@
     (property "Reference" "J20" (id 0) (at 163.83 123.19 0))
     (property "Value" "3V3" (id 1) (at 166.37 123.19 0))
-    (property "Footprint" "" (id 2) (at 166.37 127 0)
+    (property "Footprint" "Connector_PinHeader_2.54mm:PinHeader_1x05_P2.54mm_Vertical" (id 2) (at 166.37 127 0)
       (effects (font (size 1.27 1.27)) hide)
     )
@@
     (property "Reference" "J21" (id 0) (at 177.8 97.79 0))
     (property "Value" "GND" (id 1) (at 177.8 95.25 0))
-    (property "Footprint" "" (id 2) (at 181.61 95.25 0)
+    (property "Footprint" "Connector_PinHeader_2.54mm:PinHeader_1x05_P2.54mm_Vertical" (id 2) (at 181.61 95.25 0)
       (effects (font (size 1.27 1.27)) hide)
     )
@@
       (effects (font (size 1.27 1.27)) (justify left))
     )
-    (property "Footprint" "" (id 2) (at 149.86 83.82 0)
+    (property "Footprint" "Connector_PinHeader_2.54mm:PinHeader_1x13_P2.54mm_Vertical" (id 2) (at 149.86 83.82 0)
       (effects (font (size 1.27 1.27)) hide)
     )
@@
     (property "Reference" "J22" (id 0) (at 177.8 118.11 0))
     (property "Value" "5V" (id 1) (at 177.8 115.57 0))
-    (property "Footprint" "" (id 2) (at 181.61 115.57 0)
+    (property "Footprint" "Connector_PinHeader_2.54mm:PinHeader_1x05_P2.54mm_Vertical" (id 2) (at 181.61 115.57 0)
       (effects (font (size 1.27 1.27)) hide)
     )
@@
     (property "Reference" "J18" (id 0) (at 120.65 115.57 0))
     (property "Value" "SPI" (id 1) (at 120.65 118.11 0))
-    (property "Footprint" "" (id 2) (at 116.84 118.11 0)
+    (property "Footprint" "Connector_PinHeader_2.54mm:PinHeader_1x05_P2.54mm_Vertical" (id 2) (at 116.84 118.11 0)
       (effects (font (size 1.27 1.27)) hide)
     )

Commit message: did some minor stuff
Other:
- company: (none) -> Hochschule Pforzheim
- title: (none) -> eduSignal
Changed lines of the file:
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@@
 (kicad_sch (version 20211123) (generator eeschema)
   (paper "A4")
+  (title_block
+    (title "eduSignal")
+    (date "2022-07-14")
+    (rev "1")
+    (company "Hochschule Pforzheim")
+    (comment 1 "Patrick Hanner")
+    (comment 2 "Biosignal development board")
+  )
   (junction (at 187.96 113.03) (diameter 0) (color 0 0 0 0)
   )
