File: board/display.kicad_sch (KiCad schematic)
At the start: 8 parts, among them J1 Display, U12 TSC2003

Commit message: did some minor stuff
Other:
- company: (none) -> Hochschule Pforzheim
- title: (none) -> eduSignal
Changed lines of the file:
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@@
 (kicad_sch (version 20211123) (generator eeschema)
   (paper "A4")
+  (title_block
+    (title "eduSignal")
+    (date "2022-07-14")
+    (rev "1")
+    (company "Hochschule Pforzheim")
+    (comment 1 "Patrick Hanner")
+    (comment 2 "Biosignal development board")
+  )
   (no_connect (at 151.13 101.6))
   (wire (pts (xy 199.39 64.77) (xy 201.93 64.77))
