File: board/eeg_mux.kicad_sch (KiCad schematic)
At the start: 12 parts

Commit message: updated hw project
Parts:
- J?: value (none) -> Device Electrodes
- J?: value (none) -> EEG Out
- U? (x10): value (none) -> ADG733BRQ; footprint (none) -> Package_SO:QSOP-16_3.9x4.9mm_P0.635mm
Changed lines of the file:
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@@
     (in_bom yes) (on_board yes) (fields_autoplaced)
     (property "Reference" "U?" (id 0) (at 64.77 113.03 0))
-    (property "Value" "" (id 1) (at 64.77 115.57 0))
-    (property "Footprint" "" (id 2) (at 64.77 120.65 0)
+    (property "Value" "ADG733BRQ" (id 1) (at 64.77 115.57 0))
+    (property "Footprint" "Package_SO:QSOP-16_3.9x4.9mm_P0.635mm" (id 2) (at 64.77 120.65 0)
       (effects (font (size 1.27 1.27)) hide)
     )
@@
       (effects (font (size 1.27 1.27)) hide)
     )
-    (property "Value" "" (id 1) (at 203.2 96.52 0))
+    (property "Value" "VDD" (id 1) (at 203.2 96.52 0))
     (property "Footprint" "" (id 2) (at 203.2 101.6 0)
       (effects (font (size 1.27 1.27)) hide)
@@
     (in_bom yes) (on_board yes) (fields_autoplaced)
     (property "Reference" "U?" (id 0) (at 64.77 71.755 0))
-    (property "Value" "" (id 1) (at 64.77 74.295 0))
-    (property "Footprint" "" (id 2) (at 64.77 78.74 0)
+    (property "Value" "ADG733BRQ" (id 1) (at 64.77 74.295 0))
+    (property "Footprint" "Package_SO:QSOP-16_3.9x4.9mm_P0.635mm" (id 2) (at 64.77 78.74 0)
       (effects (font (size 1.27 1.27)) hide)
     )
@@
     (in_bom yes) (on_board yes) (fields_autoplaced)
     (property "Reference" "U?" (id 0) (at 64.77 92.075 0))
-    (property "Value" "" (id 1) (at 64.77 94.615 0))
-    (property "Footprint" "" (id 2) (at 64.77 99.06 0)
+    (property "Value" "ADG733BRQ" (id 1) (at 64.77 94.615 0))
+    (property "Footprint" "Package_SO:QSOP-16_3.9x4.9mm_P0.635mm" (id 2) (at 64.77 99.06 0)
       (effects (font (size 1.27 1.27)) hide)
     )
@@
       (effects (font (size 1.27 1.27)) (justify left))
     )
-    (property "Value" "" (id 1) (at 137.16 104.1399 0)
+    (property "Value" "Device Electrodes" (id 1) (at 137.16 104.1399 0)
       (effects (font (size 1.27 1.27)) (justify left))
     )
@@
       (effects (font (size 1.27 1.27)) (justify left))
     )
-    (property "Value" "" (id 1) (at 212.09 115.5699 0)
-      (effects (font (size 1.27 1.27)) (justify left))
-    )
-    (property "Footprint" "" (id 2) (at 203.2 114.3 0)
+    (property "Value" "ADG733BRQ" (id 1) (at 212.09 115.5699 0)
+      (effects (font (size 1.27 1.27)) (justify left))
+    )
+    (property "Footprint" "Package_SO:QSOP-16_3.9x4.9mm_P0.635mm" (id 2) (at 203.2 114.3 0)
       (effects (font (size 1.27 1.27)) hide)
     )
@@
     (in_bom yes) (on_board yes) (fields_autoplaced)
     (property "Reference" "U?" (id 0) (at 64.77 28.575 0))
-    (property "Value" "" (id 1) (at 64.77 31.115 0))
-    (property "Footprint" "" (id 2) (at 64.77 35.56 0)
+    (property "Value" "ADG733BRQ" (id 1) (at 64.77 31.115 0))
+    (property "Footprint" "Package_SO:QSOP-16_3.9x4.9mm_P0.635mm" (id 2) (at 64.77 35.56 0)
       (effects (font (size 1.27 1.27)) hide)
     )
@@
       (effects (font (size 1.27 1.27)) (justify left))
     )
-    (property "Value" "" (id 1) (at 240.665 115.5699 0)
-      (effects (font (size 1.27 1.27)) (justify left))
-    )
-    (property "Footprint" "" (id 2) (at 232.41 114.3 0)
+    (property "Value" "ADG733BRQ" (id 1) (at 240.665 115.5699 0)
+      (effects (font (size 1.27 1.27)) (justify left))
+    )
+    (property "Footprint" "Package_SO:QSOP-16_3.9x4.9mm_P0.635mm" (id 2) (at 232.41 114.3 0)
       (effects (font (size 1.27 1.27)) hide)
     )
@@
       (effects (font (size 1.27 1.27)) hide)
     )
-    (property "Value" "" (id 1) (at 205.74 132.08 0))
+    (property "Value" "GND" (id 1) (at 205.74 132.08 0))
     (property "Footprint" "" (id 2) (at 205.74 127 0)
       (effects (font (size 1.27 1.27)) hide)
@@
       (effects (font (size 1.27 1.27)) (justify left))
     )
-    (property "Value" "" (id 1) (at 118.11 166.3699 0)
+    (property "Value" "EEG Out" (id 1) (at 118.11 166.3699 0)
       (effects (font (size 1.27 1.27)) (justify left))
     )
@@
       (effects (font (size 1.27 1.27)) (justify left))
     )
-    (property "Value" "" (id 1) (at 237.49 77.4699 0)
-      (effects (font (size 1.27 1.27)) (justify left))
-    )
-    (property "Footprint" "" (id 2) (at 229.87 76.2 0)
+    (property "Value" "ADG733BRQ" (id 1) (at 237.49 77.4699 0)
+      (effects (font (size 1.27 1.27)) (justify left))
+    )
+    (property "Footprint" "Package_SO:QSOP-16_3.9x4.9mm_P0.635mm" (id 2) (at 229.87 76.2 0)
       (effects (font (size 1.27 1.27)) hide)
     )
@@
       (effects (font (size 1.27 1.27)) (justify left))
     )
-    (property "Value" "" (id 1) (at 212.725 77.4699 0)
-      (effects (font (size 1.27 1.27)) (justify left))
-    )
-    (property "Footprint" "" (id 2) (at 203.2 76.2 0)
+    (property "Value" "ADG733BRQ" (id 1) (at 212.725 77.4699 0)
+      (effects (font (size 1.27 1.27)) (justify left))
+    )
+    (property "Footprint" "Package_SO:QSOP-16_3.9x4.9mm_P0.635mm" (id 2) (at 203.2 76.2 0)
       (effects (font (size 1.27 1.27)) hide)
     )
@@
       (effects (font (size 1.27 1.27)) hide)
     )
-    (property "Value" "" (id 1) (at 203.2 58.42 0))
+    (property "Value" "VDD" (id 1) (at 203.2 58.42 0))
     (property "Footprint" "" (id 2) (at 203.2 63.5 0)
       (effects (font (size 1.27 1.27)) hide)
@@
     (in_bom yes) (on_board yes) (fields_autoplaced)
     (property "Reference" "U?" (id 0) (at 64.77 134.62 0))
-    (property "Value" "" (id 1) (at 64.77 137.16 0))
-    (property "Footprint" "" (id 2) (at 64.77 142.24 0)
+    (property "Value" "ADG733BRQ" (id 1) (at 64.77 137.16 0))
+    (property "Footprint" "Package_SO:QSOP-16_3.9x4.9mm_P0.635mm" (id 2) (at 64.77 142.24 0)
       (effects (font (size 1.27 1.27)) hide)
     )
@@
     (in_bom yes) (on_board yes) (fields_autoplaced)
     (property "Reference" "U?" (id 0) (at 64.77 50.165 0))
-    (property "Value" "" (id 1) (at 64.77 52.705 0))
-    (property "Footprint" "" (id 2) (at 64.77 57.15 0)
+    (property "Value" "ADG733BRQ" (id 1) (at 64.77 52.705 0))
+    (property "Footprint" "Package_SO:QSOP-16_3.9x4.9mm_P0.635mm" (id 2) (at 64.77 57.15 0)
       (effects (font (size 1.27 1.27)) hide)
     )
@@
       (effects (font (size 1.27 1.27)) hide)
     )
-    (property "Value" "" (id 1) (at 205.74 93.98 0))
+    (property "Value" "GND" (id 1) (at 205.74 93.98 0))
     (property "Footprint" "" (id 2) (at 205.74 88.9 0)
       (effects (font (size 1.27 1.27)) hide)

Commit message: updated schematic
Parts:
- removed U? (x10): ADG733BRQ, Package_SO:QSOP-16_3.9x4.9mm_P0.635mm, symbol Analog_Switch:ADG733BRQ
- added JP?: IN1N_SEL, symbol Jumper:Jumper_3_Bridged12
- added JP?: IN4N_SEL, symbol Jumper:Jumper_3_Bridged12
- added JP?: IN3N_SEL, symbol Jumper:Jumper_3_Bridged12
- added JP?: IN2N_SEL, symbol Jumper:Jumper_3_Bridged12
- J?: symbol Connector_Generic:Conn_01x05 -> Connector_Generic:Conn_01x06
Connections:
- net BIAS: now also J?.6 (Pin_6); no longer J?.5 (Pin_5)
- net IN1N: now also JP?.2 (C)
- net IN1P: now also J?.1 (Pin_1), J?.1 (Pin_1)
- net IN2N: now also JP?.2 (C)
- net IN2P: now also J?.2 (Pin_2), J?.3 (Pin_3)
- net IN3N: now also JP?.2 (C)
- net IN3P: now also J?.3 (Pin_3), J?.5 (Pin_5)
- net IN4N: now also JP?.2 (C); no longer J?.8 (Pin_8)
- net IN4P: now also J?.4 (Pin_4)
- net IN2N_OUT: now reaches J?.4 (Pin_4)
- net IN2N_OUT: now also JP?.1 (A)
- net IN1N_OUT: now reaches J?.2 (Pin_2)
- net IN1N_OUT: now also JP?.1 (A)
- net IN3N_OUT: now reaches J?.6 (Pin_6)
- net IN3N_OUT: now also JP?.1 (A)
- new net IN4N_OUT: J?.8 (Pin_8), JP?.1 (A)
- new net NCOMM: J?.5 (Pin_5), JP?.3 (B), JP?.3 (B), JP?.3 (B), JP?.3 (B)
Other:
- note added: "NCOMM Selector lets you choose between individual negative output electrodes or one single common output"
- note added: "To connect device with the internal electrodes connect IN1N and IN2N with the common electrode. Other channels are reserved for further use!"
- moved on the sheet: J?

Commit message: ERC run
Parts:
- gave numbers to parts that had none: 6
Changed lines of the file:
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@@
   (symbol (lib_id "Connector_Generic:Conn_01x06") (at 156.21 87.63 0) (unit 1)
     (in_bom yes) (on_board yes) (fields_autoplaced)
-    (property "Reference" "J?" (id 0) (at 158.75 87.6299 0)
+    (property "Reference" "J5" (id 0) (at 158.75 87.6299 0)
       (effects (font (size 1.27 1.27)) (justify left))
     )
@@
   (symbol (lib_id "Jumper:Jumper_3_Bridged12") (at 60.96 165.1 270) (unit 1)
     (in_bom yes) (on_board yes) (fields_autoplaced)
-    (property "Reference" "JP?" (id 0) (at 63.5 163.8299 90)
+    (property "Reference" "JP4" (id 0) (at 63.5 163.8299 90)
       (effects (font (size 1.27 1.27)) (justify left))
     )
@@
   (symbol (lib_id "Jumper:Jumper_3_Bridged12") (at 87.63 184.15 270) (unit 1)
     (in_bom yes) (on_board yes) (fields_autoplaced)
-    (property "Reference" "JP?" (id 0) (at 90.17 182.8799 90)
+    (property "Reference" "JP7" (id 0) (at 90.17 182.8799 90)
       (effects (font (size 1.27 1.27)) (justify left))
     )
@@
   (symbol (lib_id "Jumper:Jumper_3_Bridged12") (at 87.63 165.1 270) (unit 1)
     (in_bom yes) (on_board yes) (fields_autoplaced)
-    (property "Reference" "JP?" (id 0) (at 90.17 163.8299 90)
+    (property "Reference" "JP6" (id 0) (at 90.17 163.8299 90)
       (effects (font (size 1.27 1.27)) (justify left))
     )
@@
   (symbol (lib_id "Connector_Generic:Conn_01x09") (at 124.46 87.63 0) (unit 1)
     (in_bom yes) (on_board yes) (fields_autoplaced)
-    (property "Reference" "J?" (id 0) (at 127 87.6299 0)
+    (property "Reference" "J4" (id 0) (at 127 87.6299 0)
       (effects (font (size 1.27 1.27)) (justify left))
     )
@@
   (symbol (lib_id "Jumper:Jumper_3_Bridged12") (at 60.96 184.15 270) (unit 1)
     (in_bom yes) (on_board yes) (fields_autoplaced)
-    (property "Reference" "JP?" (id 0) (at 63.5 182.8799 90)
+    (property "Reference" "JP5" (id 0) (at 63.5 182.8799 90)
       (effects (font (size 1.27 1.27)) (justify left))
     )

Commit message: added footprints to symbols and started layout
Parts:
- J4: footprint (none) -> Connector_PinHeader_2.54mm:PinHeader_1x09_P2.54mm_Vertical
- J5: footprint (none) -> Connector_PinHeader_2.54mm:PinHeader_1x06_P2.54mm_Vertical
- JP4, JP5, JP6, JP7: footprint (none) -> Connector_PinHeader_2.54mm:PinHeader_1x03_P2.54mm_Vertical
Changed lines of the file:
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@@
       (effects (font (size 1.27 1.27)) (justify left))
     )
-    (property "Footprint" "" (id 2) (at 156.21 87.63 0)
+    (property "Footprint" "Connector_PinHeader_2.54mm:PinHeader_1x06_P2.54mm_Vertical" (id 2) (at 156.21 87.63 0)
       (effects (font (size 1.27 1.27)) hide)
     )
@@
       (effects (font (size 1.27 1.27)) (justify left))
     )
-    (property "Footprint" "" (id 2) (at 60.96 165.1 0)
+    (property "Footprint" "Connector_PinHeader_2.54mm:PinHeader_1x03_P2.54mm_Vertical" (id 2) (at 60.96 165.1 0)
       (effects (font (size 1.27 1.27)) hide)
     )
@@
       (effects (font (size 1.27 1.27)) (justify left))
     )
-    (property "Footprint" "" (id 2) (at 87.63 184.15 0)
+    (property "Footprint" "Connector_PinHeader_2.54mm:PinHeader_1x03_P2.54mm_Vertical" (id 2) (at 87.63 184.15 0)
       (effects (font (size 1.27 1.27)) hide)
     )
@@
       (effects (font (size 1.27 1.27)) (justify left))
     )
-    (property "Footprint" "" (id 2) (at 87.63 165.1 0)
+    (property "Footprint" "Connector_PinHeader_2.54mm:PinHeader_1x03_P2.54mm_Vertical" (id 2) (at 87.63 165.1 0)
       (effects (font (size 1.27 1.27)) hide)
     )
@@
       (effects (font (size 1.27 1.27)) (justify left))
     )
-    (property "Footprint" "" (id 2) (at 124.46 87.63 0)
+    (property "Footprint" "Connector_PinHeader_2.54mm:PinHeader_1x09_P2.54mm_Vertical" (id 2) (at 124.46 87.63 0)
       (effects (font (size 1.27 1.27)) hide)
     )
@@
       (effects (font (size 1.27 1.27)) (justify left))
     )
-    (property "Footprint" "" (id 2) (at 60.96 184.15 0)
+    (property "Footprint" "Connector_PinHeader_2.54mm:PinHeader_1x03_P2.54mm_Vertical" (id 2) (at 60.96 184.15 0)
       (effects (font (size 1.27 1.27)) hide)
     )

Commit message: WIP pushed for meeting
Connections:
- net IN2N_OUT: now also JP5.1 (A); no longer JP6.1 (A)
- net IN3N_OUT: now also JP6.1 (A); no longer JP5.1 (A)
Changed lines of the file:
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@@
     (effects (font (size 1.27 1.27)) (justify right bottom))
   )
-  (label "IN2N_OUT" (at 87.63 158.75 0)
+  (label "IN2N_OUT" (at 60.96 177.8 0)
     (effects (font (size 1.27 1.27)) (justify left bottom))
   )
@@
     (effects (font (size 1.27 1.27)) (justify left bottom))
   )
-  (label "IN3N_OUT" (at 60.96 177.8 0)
+  (label "IN3N_OUT" (at 87.63 158.75 0)
     (effects (font (size 1.27 1.27)) (justify left bottom))
   )

Commit message: did some minor stuff
Other:
- company: (none) -> Hochschule Pforzheim
- title: (none) -> eduSignal
Changed lines of the file:
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@@
 (kicad_sch (version 20211123) (generator eeschema)
   (paper "A4")
+  (title_block
+    (title "eduSignal")
+    (date "2022-07-14")
+    (rev "1")
+    (company "Hochschule Pforzheim")
+    (comment 1 "Patrick Hanner")
+    (comment 2 "Biosignal development board")
+  )
   (polyline (pts (xy 12.7 146.05) (xy 106.68 146.05))
     (stroke (width 0) (type default) (color 0 0 0 0))
