File: board/io_extender.kicad_sch (KiCad schematic)
At the start: 3 parts

Commit message: ERC run
Parts:
- added JP10: A1, symbol Jumper:Jumper_3_Bridged12
- added JP11: A2, symbol Jumper:Jumper_3_Bridged12
- added JP12: A0, symbol Jumper:Jumper_3_Bridged12
- gave numbers to parts that had none: 3
Connections:
- net 3V3: now also JP10.3 (B), JP11.3 (B), JP12.3 (B)
- net GND: now also JP10.1 (A), JP11.1 (A), JP12.1 (A)
- net at U11.1 (A0): now also JP12.2 (C)
- net P5: now reaches U11.10 (P5)
- net P6: now reaches U11.11 (P6)
- net P7: now reaches U11.12 (P7)
- net at U11.2 (A1): now also JP11.2 (C)
- net at U11.3 (A2): now also JP10.2 (C)
- net P0: now reaches U11.4 (P0)
- net P1: now reaches U11.5 (P1)
- net P2: now reaches U11.6 (P2)
- net P3: now reaches U11.7 (P3)
- net P4: now reaches U11.9 (P4)
Other:
- moved on the sheet: C46, C47, U11

Commit message: updated schematic after review
Other:
- note added: "Adress: (default) Write 0x40 Read 0x41"
Changed lines of the file:
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@@
     (stroke (width 0) (type default) (color 0 0 0 0))
+  )
+  (text "Adress: (default)\nWrite 0x40\nRead  0x41" (at 133.35 107.95 0)
+    (effects (font (size 1.27 1.27)) (justify left bottom))
   )
   (hierarchical_label "P2" (shape bidirectional) (at 184.15 88.9 0)

Commit message: added footprints to symbols and started layout
Parts:
- C46: footprint (none) -> Capacitor_SMD:C_0603_1608Metric
- C47: footprint (none) -> Capacitor_SMD:C_0402_1005Metric
- JP10, JP11, JP12: footprint (none) -> Jumper:SolderJumper-3_P1.3mm_Bridged12_Pad1.0x1.5mm
- U11: footprint (none) -> Package_SO:SOIC-16W_7.5x10.3mm_P1.27mm
Changed lines of the file:
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@@
       (effects (font (size 1.27 1.27)) (justify left))
     )
-    (property "Footprint" "" (id 2) (at 109.22 120.65 0)
+    (property "Footprint" "Capacitor_SMD:C_0603_1608Metric" (id 2) (at 109.22 120.65 0)
       (effects (font (size 1.27 1.27)) hide)
     )
@@
       (effects (font (size 1.27 1.27)) (justify left))
     )
-    (property "Footprint" "" (id 2) (at 171.45 93.98 0)
+    (property "Footprint" "Package_SO:SOIC-16W_7.5x10.3mm_P1.27mm" (id 2) (at 171.45 93.98 0)
       (effects (font (size 1.27 1.27)) hide)
     )
@@
     (property "Reference" "JP11" (id 0) (at 118.11 77.47 0))
     (property "Value" "A2" (id 1) (at 118.11 80.01 0))
-    (property "Footprint" "" (id 2) (at 118.11 83.82 0)
+    (property "Footprint" "Jumper:SolderJumper-3_P1.3mm_Bridged12_Pad1.0x1.5mm" (id 2) (at 118.11 83.82 0)
       (effects (font (size 1.27 1.27)) hide)
     )
@@
     (property "Reference" "JP12" (id 0) (at 135.89 77.47 0))
     (property "Value" "A0" (id 1) (at 135.89 80.01 0))
-    (property "Footprint" "" (id 2) (at 135.89 83.82 0)
+    (property "Footprint" "Jumper:SolderJumper-3_P1.3mm_Bridged12_Pad1.0x1.5mm" (id 2) (at 135.89 83.82 0)
       (effects (font (size 1.27 1.27)) hide)
     )
@@
     (property "Reference" "JP10" (id 0) (at 99.06 77.47 0))
     (property "Value" "A1" (id 1) (at 99.06 80.01 0))
-    (property "Footprint" "" (id 2) (at 99.06 83.82 0)
+    (property "Footprint" "Jumper:SolderJumper-3_P1.3mm_Bridged12_Pad1.0x1.5mm" (id 2) (at 99.06 83.82 0)
       (effects (font (size 1.27 1.27)) hide)
     )
@@
       (effects (font (size 1.27 1.27)) (justify left))
     )
-    (property "Footprint" "" (id 2) (at 119.38 120.65 0)
+    (property "Footprint" "Capacitor_SMD:C_0402_1005Metric" (id 2) (at 119.38 120.65 0)
       (effects (font (size 1.27 1.27)) hide)
     )

Commit message: did some minor stuff
Other:
- company: (none) -> Hochschule Pforzheim
- title: (none) -> eduSignal
Changed lines of the file:
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@@
 (kicad_sch (version 20211123) (generator eeschema)
   (paper "A4")
+  (title_block
+    (title "eduSignal")
+    (date "2022-07-14")
+    (rev "1")
+    (company "Hochschule Pforzheim")
+    (comment 1 "Patrick Hanner")
+    (comment 2 "Biosignal development board")
+  )
   (junction (at 109.22 124.46) (diameter 0) (color 0 0 0 0)
   )
