File: board/ekg.kicad_sch (KiCad schematic)
At the start: 35 parts, among them J2 BIAS, J3 SRB, U2 ADS1299-x

Commit message: WIP pushed for meeting
Parts:
- removed C6: 1u, Capacitor_SMD:C_0603_1608Metric, symbol Device:C_Small
Changed lines of the file:
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@@
   (junction (at 82.55 36.83) (diameter 0) (color 0 0 0 0)
   )
-  (junction (at 100.33 50.8) (diameter 0) (color 0 0 0 0)
-  )
   (junction (at 66.675 161.29) (diameter 0) (color 0 0 0 0)
   )
@@
   )
   (junction (at 158.75 69.85) (diameter 0) (color 0 0 0 0)
-  )
-  (junction (at 100.33 44.45) (diameter 0) (color 0 0 0 0)
   )
   (no_connect (at 121.92 120.65))
@@
     (stroke (width 0) (type default) (color 0 0 0 0))
   )
-  (wire (pts (xy 107.95 44.45) (xy 100.33 44.45))
-    (stroke (width 0) (type default) (color 0 0 0 0))
-  )
   (wire (pts (xy 74.93 62.23) (xy 82.55 62.23))
     (stroke (width 0) (type default) (color 0 0 0 0))
   )
-  (wire (pts (xy 100.33 44.45) (xy 100.33 45.72))
-    (stroke (width 0) (type default) (color 0 0 0 0))
-  )
   (wire (pts (xy 100.33 50.8) (xy 100.33 52.07))
     (stroke (width 0) (type default) (color 0 0 0 0))
@@
     (stroke (width 0) (type default) (color 0 0 0 0))
   )
-  (wire (pts (xy 95.25 44.45) (xy 100.33 44.45))
+  (wire (pts (xy 95.25 44.45) (xy 107.95 44.45))
     (stroke (width 0) (type default) (color 0 0 0 0))
   )
@@
     (pin "1")
   )
-  (symbol (lib_id "Device:C_Small") (at 100.33 48.26 0) (unit 1)
-    (in_bom yes) (on_board yes) (fields_autoplaced)
-    (property "Reference" "C6" (id 0) (at 102.87 46.9962 0)
-      (effects (font (size 1.27 1.27)) (justify left))
-    )
-    (property "Value" "1u" (id 1) (at 102.87 49.5362 0)
-      (effects (font (size 1.27 1.27)) (justify left))
-    )
-    (property "Footprint" "Capacitor_SMD:C_0603_1608Metric" (id 2) (at 100.33 48.26 0)
-      (effects (font (size 1.27 1.27)) hide)
-    )
-    (property "Datasheet" "~" (id 3) (at 100.33 48.26 0)
-      (effects (font (size 1.27 1.27)) hide)
-    )
-    (pin "1")
-    (pin "2")
-  )
   (symbol (lib_id "ownLib:ADS1299-x") (at 135.89 91.44 0) (unit 1)

Commit message: finished layout for review
Parts:
- JP1: value BIASOUT SEL -> FILTER OUT
Connections:
- net at U2.27 (NC): no longer U2.29 (NC)
Changed lines of the file:
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@@
   (symbol (lib_id "Jumper:Jumper_3_Bridged12") (at 41.91 172.72 0) (mirror y) (unit 1)
     (in_bom yes) (on_board yes) (fields_autoplaced)
-    (property "Reference" "JP1" (id 0) (at 41.91 167.005 0))
-    (property "Value" "BIASOUT SEL" (id 1) (at 41.91 169.545 0))
+    (property "Reference" "JP1" (id 0) (at 41.91 166.37 0))
+    (property "Value" "FILTER OUT" (id 1) (at 41.91 168.91 0))
     (property "Footprint" "Connector_PinHeader_2.54mm:PinHeader_1x03_P2.54mm_Vertical" (id 2) (at 41.91 172.72 0)
       (effects (font (size 1.27 1.27)) hide)

Commit message: did some minor stuff
Other:
- company: (none) -> Hochschule Pforzheim
- title: (none) -> eduSignal
Changed lines of the file:
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@@
 (kicad_sch (version 20211123) (generator eeschema)
   (paper "A4")
+  (title_block
+    (title "eduSignal")
+    (date "2022-07-14")
+    (rev "1")
+    (company "Hochschule Pforzheim")
+    (comment 1 "Patrick Hanner")
+    (comment 2 "Biosignal development board")
+  )
   (junction (at 158.75 90.17) (diameter 0) (color 0 0 0 0)
   )

Commit message: worked feedback into layout with dp
Connections:
- net +3V3: no longer C11.1, U2.19 (AVDD), U2.21 (AVDD), U2.22 (AVDD), U2.56 (AVDD), U2.59 (AVDD)
- net +5VA: now also C11.1, U2.19 (AVDD), U2.21 (AVDD), U2.22 (AVDD), U2.56 (AVDD), U2.59 (AVDD)
Changed lines of the file:
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@@
     (pin "2")
+  )
+  (symbol (lib_id "power:+5VA") (at 115.57 40.64 90) (unit 1)
+    (in_bom yes) (on_board yes) (fields_autoplaced)
+    (property "Reference" "#PWR0104" (id 0) (at 119.38 40.64 0)
+      (effects (font (size 1.27 1.27)) hide)
+    )
+    (property "Value" "+5VA" (id 1) (at 111.76 40.6399 90)
+      (effects (font (size 1.27 1.27)) (justify left))
+    )
+    (property "Footprint" "" (id 2) (at 115.57 40.64 0)
+      (effects (font (size 1.27 1.27)) hide)
+    )
+    (property "Datasheet" "" (id 3) (at 115.57 40.64 0)
+      (effects (font (size 1.27 1.27)) hide)
+    )
+    (pin "1")
   )
   (symbol (lib_id "Device:C_Small") (at 87.63 66.04 270) (unit 1)
@@
       (effects (font (size 1.27 1.27)) hide)
     )
-    (pin "1")
-  )
-  (symbol (lib_id "power:+3V3") (at 115.57 40.64 90) (unit 1)
-    (in_bom yes) (on_board yes) (fields_autoplaced)
-    (property "Reference" "#PWR013" (id 0) (at 119.38 40.64 0)
-      (effects (font (size 1.27 1.27)) hide)
-    )
-    (property "Value" "+3V3" (id 1) (at 111.76 40.6399 90)
-      (effects (font (size 1.27 1.27)) (justify left))
-    )
-    (property "Footprint" "" (id 2) (at 115.57 40.64 0)
-      (effects (font (size 1.27 1.27)) hide)
-    )
-    (property "Datasheet" "" (id 3) (at 115.57 40.64 0)
-      (effects (font (size 1.27 1.27)) hide)
-    )
