File: board/pulsoxy.kicad_sch (KiCad schematic)
At the start: 2 parts

Commit message: updated schematic
Connections:
- net +3V3 renamed 3V3
- net +5V renamed 5V
Changed lines of the file:
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@@
     (effects (font (size 1.27 1.27)) (justify right))
+  )
+  (hierarchical_label "5V" (shape input) (at 143.51 81.28 90)
+    (effects (font (size 1.27 1.27)) (justify left))
   )
   (hierarchical_label "SDA" (shape bidirectional) (at 135.89 93.98 180)
     (effects (font (size 1.27 1.27)) (justify right))
+  )
+  (hierarchical_label "3V3" (shape input) (at 125.73 81.28 90)
+    (effects (font (size 1.27 1.27)) (justify left))
   )
   (symbol (lib_id "Jumper:Jumper_3_Bridged12") (at 134.62 82.55 0) (unit 1)
@@
       (effects (font (size 1.27 1.27)) hide)
     )
-    (pin "1")
-  )
-  (symbol (lib_id "power:+3V3") (at 125.73 81.28 0) (unit 1)
-    (in_bom yes) (on_board yes) (fields_autoplaced)
-    (property "Reference" "#PWR?" (id 0) (at 125.73 85.09 0)
-      (effects (font (size 1.27 1.27)) hide)
-    )
-    (property "Value" "+3V3" (id 1) (at 125.73 76.2 0))
-    (property "Footprint" "" (id 2) (at 125.73 81.28 0)
-      (effects (font (size 1.27 1.27)) hide)
-    )
-    (property "Datasheet" "" (id 3) (at 125.73 81.28 0)
-      (effects (font (size 1.27 1.27)) hide)
-    )
-    (pin "1")
-  )
-  (symbol (lib_id "power:+5V") (at 143.51 81.28 0) (unit 1)
-    (in_bom yes) (on_board yes) (fields_autoplaced)
-    (property "Reference" "#PWR?" (id 0) (at 143.51 85.09 0)
-      (effects (font (size 1.27 1.27)) hide)
-    )
-    (property "Value" "+5V" (id 1) (at 143.51 76.2 0))
-    (property "Footprint" "" (id 2) (at 143.51 81.28 0)
-      (effects (font (size 1.27 1.27)) hide)
-    )
-    (property "Datasheet" "" (id 3) (at 143.51 81.28 0)
-      (effects (font (size 1.27 1.27)) hide)
-    )

Commit message: added io expander
Other:
- note added: "Address: Read: AE Write: AF"
Changed lines of the file:
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@@
     (stroke (width 0) (type default) (color 0 0 0 0))
+  )
+  (text "Address:\nRead: AE\nWrite: AF" (at 153.67 93.98 0)
+    (effects (font (size 1.27 1.27)) (justify left bottom))
   )
   (hierarchical_label "SCL" (shape bidirectional) (at 135.89 96.52 180)

Commit message: ERC run
Parts:
- gave numbers to parts that had none: 2
Changed lines of the file:
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@@
   (symbol (lib_id "Jumper:Jumper_3_Bridged12") (at 134.62 82.55 0) (unit 1)
     (in_bom yes) (on_board yes) (fields_autoplaced)
-    (property "Reference" "JP?" (id 0) (at 134.62 76.2 0))
+    (property "Reference" "JP9" (id 0) (at 134.62 76.2 0))
     (property "Value" "VCC_SEL" (id 1) (at 134.62 78.74 0))
     (property "Footprint" "" (id 2) (at 134.62 82.55 0)
@@
   (symbol (lib_id "Connector_Generic:Conn_01x04") (at 140.97 96.52 0) (mirror x) (unit 1)
     (in_bom yes) (on_board yes) (fields_autoplaced)
-    (property "Reference" "J?" (id 0) (at 140.97 85.09 0))
+    (property "Reference" "J16" (id 0) (at 140.97 85.09 0))
     (property "Value" "Conn_01x04" (id 1) (at 140.97 87.63 0))
     (property "Footprint" "" (id 2) (at 140.97 96.52 0)
@@
   (symbol (lib_id "power:GND") (at 134.62 100.33 0) (unit 1)
     (in_bom yes) (on_board yes) (fields_autoplaced)
-    (property "Reference" "#PWR?" (id 0) (at 134.62 106.68 0)
+    (property "Reference" "#PWR063" (id 0) (at 134.62 106.68 0)
       (effects (font (size 1.27 1.27)) hide)
     )

Commit message: updated schematic after review
Parts:
- J16: value Conn_01x04 -> OXY
Changed lines of the file:
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@@
     (in_bom yes) (on_board yes) (fields_autoplaced)
     (property "Reference" "J16" (id 0) (at 140.97 85.09 0))
-    (property "Value" "Conn_01x04" (id 1) (at 140.97 87.63 0))
+    (property "Value" "OXY" (id 1) (at 140.97 87.63 0))
     (property "Footprint" "" (id 2) (at 140.97 96.52 0)
       (effects (font (size 1.27 1.27)) hide)

Commit message: added footprints to symbols and started layout
Parts:
- J16: footprint (none) -> Connector_PinHeader_2.54mm:PinHeader_1x04_P2.54mm_Vertical
- JP9: footprint (none) -> Jumper:SolderJumper-3_P1.3mm_Bridged12_Pad1.0x1.5mm
Changed lines of the file:
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@@
     (property "Reference" "JP9" (id 0) (at 134.62 76.2 0))
     (property "Value" "VCC_SEL" (id 1) (at 134.62 78.74 0))
-    (property "Footprint" "" (id 2) (at 134.62 82.55 0)
+    (property "Footprint" "Jumper:SolderJumper-3_P1.3mm_Bridged12_Pad1.0x1.5mm" (id 2) (at 134.62 82.55 0)
       (effects (font (size 1.27 1.27)) hide)
     )
@@
     (property "Reference" "J16" (id 0) (at 140.97 85.09 0))
     (property "Value" "OXY" (id 1) (at 140.97 87.63 0))
-    (property "Footprint" "" (id 2) (at 140.97 96.52 0)
+    (property "Footprint" "Connector_PinHeader_2.54mm:PinHeader_1x04_P2.54mm_Vertical" (id 2) (at 140.97 96.52 0)
       (effects (font (size 1.27 1.27)) hide)
     )

Commit message: did some minor stuff
Other:
- company: (none) -> Hochschule Pforzheim
- title: (none) -> eduSignal
Changed lines of the file:
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@@
 (kicad_sch (version 20211123) (generator eeschema)
   (paper "A4")
+  (title_block
+    (title "eduSignal")
+    (date "2022-07-14")
+    (rev "1")
+    (company "Hochschule Pforzheim")
+    (comment 1 "Patrick Hanner")
+    (comment 2 "Biosignal development board")
+  )
   (wire (pts (xy 125.73 82.55) (xy 128.27 82.55))
     (stroke (width 0) (type default) (color 0 0 0 0))

Commit message: fixed errors in schematic
Other:
- note added: "Address: Read: AF Write: AE"
- note removed: "Address: Read: AE Write: AF"
Changed lines of the file:
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@@
     (stroke (width 0) (type default) (color 0 0 0 0))
   )
-  (text "Address:\nRead: AE\nWrite: AF" (at 153.67 93.98 0)
+  (text "Address:\nRead: AF\nWrite: AE" (at 153.67 93.98 0)
     (effects (font (size 1.27 1.27)) (justify left bottom))
   )
